File: caps/z80ram/z80ram.kicad_sch (KiCad schematic)
At the start: 19 parts, among them J10 PORTG, J2 PORTA, J3 PORTB, J5 PORTD, J6 PORTE, J7 PORTF, U1 74HCT257, U2 AS6C4008-55PCN, U3 74HCT574, U4 Z80CPU

Commit message: Add reset and halt buttons to Z80 cap
Parts:
- added SW1: RESET, Button_Switch_THT:SW_PUSH_6mm, symbol Switch:SW_Push
- added SW2: HALT, Button_Switch_THT:SW_PUSH_6mm, symbol Switch:SW_Push
Connections:
- net GND: now also SW1.1, SW2.1
- net PA4: now also SW2.2
- net PB4: now also SW1.2
