File: avrbrain.kicad_pcb (KiCad board)
At the start: 4 copper layers, 85 x 56 mm, 64 parts, among them J1 UPDI, J10 PORTG, J11 UEXT, J12 SM04B-SRSS-TB, J2 PORTA, J3 PORTB, J4 PORTC, J5 PORTD, J6 PORTE, J7 PORTF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

Commit message: Add LCSC part numbers
Parts:
- C16, C17, C18, C19: footprint Capacitor_SMD:C_1206_3216Metric -> Capacitor_SMD:C_0402_1005Metric
- D2: footprint LED_SMD:LED_0805_2012Metric -> LED_SMD:LED_0603_1608Metric
- moved C17 0.98 mm to (166.6, 100.2)
- moved C16 0.94 mm to (164.6, 117.8)
- moved C19 0.85 mm to (172.9, 110.0)
- moved C18 0.67 mm to (155.4, 106.0)
- moved D2 0.20 mm to (175.1, 85.1)
Routing:
- net GND: track 49.1 -> 43.1 mm
- net +5V: track 23.6 -> 19.0 mm
- net /PB7: track 48.1 -> 45.0 mm
- net /PB6: track 49.6 -> 46.7 mm
- net /PB5: track 45.0 -> 42.3 mm
- net MISO: track 66.3 -> 63.6 mm
- net /PB4: track 46.5 -> 43.9 mm
- net /PB3: track 41.9 -> 39.5 mm
- net /PB2: track 43.3 -> 41.2 mm
- net /PB1: track 38.4 -> 36.4 mm
- net SCK: track 70.4 -> 68.4 mm
- net /PB0: track 39.2 -> 37.3 mm
- net MOSI: track 78.5 -> 76.7 mm
- net +3.3V: track 4.67 -> 3.28 mm
- net /PG4: track 27.0 -> 25.7 mm
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
Commit message: Final tweaks after uploading to JLC
Parts:
- C13: footprint Capacitor_SMD:C_0603_1608Metric_Pad1.08x0.95mm_HandSolder -> Capacitor_SMD:C_0603_1608Metric
- D1, D3, D4: footprint Diode_SMD:D_SOD-323_HandSoldering -> Diode_SMD:D_SOD-323
Routing:
- net +3.3V: track 3.28 -> 11.4 mm, vias 0 -> 4
- net GND: vias 54 -> 58
