File: avrbrain.kicad_sch (KiCad schematic)
At the start: 28 parts, among them J1 UPDI, J10 PORTG, J2 PORTA, J3 PORTB, J4 PORTC, J5 PORTD, J6 PORTE, J7 PORTF, SW1 RESET, U1 AVR128DB64x-xPT, U2 AMS1117-3.3

Commit message: Add LCSC part numbers
Parts:
- C1, C2, C3, C4, C5: LCSC part number (none) -> C1525
- C12, C7: LCSC part number (none) -> C52923
- C15, C6: LCSC part number (none) -> C12891
- C16, C17, C18, C19: footprint Capacitor_SMD:C_1206_3216Metric -> Capacitor_SMD:C_0402_1005Metric; LCSC part number (none) -> C52923
Changed lines of the file:
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@@
+			)
+		)
+		(property "LCSC part number" "C1525"
+			(at 88.9 62.23 0)
+			(effects
+				(font
+					(size 1.27 1.27)
+				)
+				(hide yes)
 			)
 		)
@@
 			)
 		)
+		(property "LCSC part number" "C1525"
+			(at 35.56 62.23 0)
+			(effects
+				(font
+					(size 1.27 1.27)
+				)
+				(hide yes)
+			)
+		)
 		(pin "1"
 		)
@@
 		)
 		(property "Description" ""
+			(at 162.56 109.22 0)
+			(effects
+				(font
+					(size 1.27 1.27)
+				)
+				(hide yes)
+			)
+		)
+		(property "LCSC part number" "C1525"
 			(at 162.56 109.22 0)
 			(effects
@@
 			)
 		)
+		(property "LCSC part number" "C52923"
+			(at 214.63 74.93 0)
+			(effects
+				(font
+					(size 1.27 1.27)
+				)
+				(hide yes)
+			)
+		)
 		(pin "1"
 		)
@@
 			)
 		)
-		(property "Footprint" "Capacitor_SMD:C_1206_3216Metric"
+		(property "Footprint" "Capacitor_SMD:C_0402_1005Metric"
 			(at 100.33 62.23 0)
 			(effects
@@
 		)
 		(property "Description" ""
+			(at 100.33 62.23 0)
+			(effects
+				(font
+					(size 1.27 1.27)
+				)
+				(hide yes)
+			)
+		)
+		(property "LCSC part number" "C52923"
 			(at 100.33 62.23 0)
 			(effects
@@
 			)
 		)
+		(property "LCSC part number" "C1525"
+			(at 76.2 62.23 0)
+			(effects
+				(font
+					(size 1.27 1.27)
+				)
+				(hide yes)
+			)
+		)
 		(pin "1"
 		)
@@
 			)
 		)
-		(property "Footprint" "Capacitor_SMD:C_1206_3216Metric"
+		(property "Footprint" "Capacitor_SMD:C_0402_1005Metric"
 			(at 45.72 62.23 0)
 			(effects
@@
 		)
 		(property "Description" ""
+			(at 45.72 62.23 0)
+			(effects
+				(font
+					(size 1.27 1.27)
+				)
+				(hide yes)
+			)
+		)
+		(property "LCSC part number" "C52923"
 			(at 45.72 62.23 0)
 			(effects
@@
 			)
 		)
+		(property "LCSC part number" "C12891"
+			(at 205.105 74.93 0)
+			(effects
+				(font
+					(size 1.27 1.27)
+				)
+				(hide yes)
+			)
+		)
 		(pin "1"
 		)
@@
 		)
 		(property "Description" ""
+			(at 254 74.93 0)
+			(effects
+				(font
+					(size 1.27 1.27)
+				)
+				(hide yes)
+			)
+		)
+		(property "LCSC part number" "C12891"
 			(at 254 74.93 0)
 			(effects
@@
 			)
 		)
-		(property "Footprint" "Capacitor_SMD:C_1206_3216Metric"
+		(property "Footprint" "Capacitor_SMD:C_0402_1005Metric"
 			(at 66.04 62.23 0)
 			(effects
@@
 		)
 		(property "Description" ""
+			(at 66.04 62.23 0)
+			(effects
+				(font
+					(size 1.27 1.27)
+				)
+				(hide yes)
+			)
+		)
+		(property "LCSC part number" "C52923"
 			(at 66.04 62.23 0)
 			(effects
@@
 			)
 		)
+		(property "LCSC part number" "C52923"
+			(at 243.84 74.93 0)
+			(effects
+				(font
+					(size 1.27 1.27)
+				)
+				(hide yes)
+			)
+		)
 		(pin "1"
 		)
@@
 			)
 		)
+		(property "LCSC part number" "C1525"
+			(at 55.88 62.23 0)
+			(effects
+				(font
+					(size 1.27 1.27)
+				)
+				(hide yes)
+			)
+		)
 		(pin "1"
 		)
@@
 			)
 		)
-		(property "Footprint" "Capacitor_SMD:C_1206_3216Metric"
+		(property "Footprint" "Capacitor_SMD:C_0402_1005Metric"
 			(at 25.4 62.23 0)
 			(effects
@@
 			(at 25.4 62.23 0)
 			(effects
+				(font
+					(size 1.27 1.27)
+				)
+				(hide yes)
+			)
+		)
+		(property "LCSC part number" "C52923"
+			(at 25.4 62.23 0)
+			(effects

Commit message: Fix LCSC field name, gerber settings
Parts:
- C1, C2, C3, C4, C5: LCSC (none) -> C1525; LCSC part number C1525 -> (none)
- C12, C16, C17, C18, C19, C7: LCSC (none) -> C52923; LCSC part number C52923 -> (none)
- C15, C6: LCSC (none) -> C12891; LCSC part number C12891 -> (none)
- U1: LCSC (none) -> C3228380
- U2: LCSC (none) -> C6186
Changed lines of the file:
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@@
 			)
 		)
-		(property "LCSC part number" "C1525"
+		(property "LCSC" "C1525"
 			(at 88.9 62.23 0)
 			(effects
@@
 			)
 		)
-		(property "LCSC part number" "C1525"
+		(property "LCSC" "C1525"
 			(at 35.56 62.23 0)
 			(effects
@@
 			)
 		)
-		(property "LCSC part number" "C1525"
+		(property "LCSC" "C1525"
 			(at 162.56 109.22 0)
 			(effects
@@
 			)
 		)
-		(property "LCSC part number" "C52923"
+		(property "LCSC" "C52923"
 			(at 214.63 74.93 0)
 			(effects
@@
 			)
 		)
+		(property "LCSC" "C3228380"
+			(at 82.55 121.92 0)
+			(effects
+				(font
+					(size 1.27 1.27)
+				)
+				(hide yes)
+			)
+		)
 		(pin "1"
 		)
@@
 			)
 		)
-		(property "LCSC part number" "C52923"
+		(property "LCSC" "C52923"
 			(at 100.33 62.23 0)
 			(effects
@@
 			)
 		)
-		(property "LCSC part number" "C1525"
+		(property "LCSC" "C1525"
 			(at 76.2 62.23 0)
 			(effects
@@
 			)
 		)
-		(property "LCSC part number" "C52923"
+		(property "LCSC" "C52923"
 			(at 45.72 62.23 0)
 			(effects
@@
 			)
 		)
-		(property "LCSC part number" "C12891"
+		(property "LCSC" "C12891"
 			(at 205.105 74.93 0)
 			(effects
@@
 			)
 		)
-		(property "LCSC part number" "C12891"
+		(property "LCSC" "C12891"
 			(at 254 74.93 0)
 			(effects
@@
 			)
 		)
-		(property "LCSC part number" "C52923"
+		(property "LCSC" "C52923"
 			(at 66.04 62.23 0)
 			(effects
@@
 			)
 		)
-		(property "LCSC part number" "C52923"
+		(property "LCSC" "C52923"
 			(at 243.84 74.93 0)
 			(effects
@@
 			)
 		)
-		(property "LCSC part number" "C1525"
+		(property "LCSC" "C1525"
 			(at 55.88 62.23 0)
 			(effects
@@
 			)
 		)
+		(property "LCSC" "C6186"
+			(at 232.41 68.58 0)
+			(effects
+				(font
+					(size 1.27 1.27)
+				)
+				(hide yes)
+			)
+		)
 		(pin "1"
 		)
@@
 			)
 		)
-		(property "LCSC part number" "C52923"
+		(property "LCSC" "C52923"
 			(at 25.4 62.23 0)
 			(effects

Commit message: Final tweaks after uploading to JLC
Parts:
- C12, C7: LCSC C52923 -> C1848
Changed lines of the file:
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@@
 			)
 		)
-		(property "LCSC" "C52923"
+		(property "LCSC" "C1848"
 			(at 214.63 74.93 0)
 			(effects
@@
 			)
 		)
-		(property "LCSC" "C52923"
+		(property "LCSC" "C1848"
 			(at 243.84 74.93 0)
 			(effects
