File: peripherals.kicad_sch (KiCad schematic)
At the start: 36 parts, among them J11 UEXT, J12 SM04B-SRSS-TB, J8 XKTF-0803-0, J9 U254-051T-4BH81-S2S, Q1 BSS138, SW3 PROG_EN, U3 CH340C, U4 PCF8563T, Y1 32kHz

Commit message: Fix LCSC field name, gerber settings
Parts:
- C1: LCSC (none) -> C107045; LCSC part number C107045 -> (none)
- C3, C8, C9: LCSC (none) -> C1525; LCSC part number C1525 -> (none)
- D1, D3, D4: LCSC (none) -> C64886; LCSC part number C64886 -> (none)
- D2: LCSC (none) -> C2286; LCSC part number C2286 -> (none)
- J12: LCSC (none) -> C160404; LCSC part number C160404 -> (none)
- J8: LCSC (none) -> C381083; LCSC part number C381083 -> (none)
- J9: LCSC (none) -> C381144; LCSC part number C381144 -> (none)
- Q1: LCSC (none) -> C7420339; LCSC part number C7420339 -> (none)
- R1, R2: LCSC (none) -> C11702; LCSC part number C11702 -> (none)
- R3, R4: LCSC (none) -> C25879; LCSC part number C25879 -> (none)
- R3, R4, R5, R6: LCSC (none) -> C25741; LCSC part number C25741 -> (none)
- U3: LCSC (none) -> C7464026; LCSC part number C7464026 -> (none)
- U4: LCSC (none) -> C7440
- Y1: LCSC (none) -> C32346; LCSC part number C32346 -> (none)
Changed lines of the file:
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@@
 			)
 		)
-		(property "LCSC part number" "C1525"
+		(property "LCSC" "C1525"
 			(at 108.585 34.925 90)
 			(effects
@@
 			)
 		)
-		(property "LCSC part number" "C1525"
+		(property "LCSC" "C1525"
 			(at 97.155 34.925 90)
 			(effects
@@
 			)
 		)
-		(property "LCSC part number" "C107045"
+		(property "LCSC" "C107045"
 			(at 110.49 156.21 0)
 			(effects
@@
 			)
 		)
-		(property "LCSC part number" "C64886"
+		(property "LCSC" "C64886"
 			(at 40.64 48.26 90)
 			(effects
@@
 			)
 		)
+		(property "LCSC" "C7440"
+			(at 88.9 156.21 0)
+			(effects
+				(font
+					(size 1.27 1.27)
+				)
+				(hide yes)
+			)
+		)
 		(pin "1"
 		)
@@
 			)
 		)
-		(property "LCSC part number" "C25879"
+		(property "LCSC" "C25879"
 			(at 45.72 145.415 0)
 			(effects
@@
 			)
 		)
-		(property "LCSC part number" "C2286"
+		(property "LCSC" "C2286"
 			(at 191.135 35.56 90)
 			(effects
@@
 			)
 		)
-		(property "LCSC part number" "C64886"
+		(property "LCSC" "C64886"
 			(at 128.905 134.62 90)
 			(effects
@@
 			)
 		)
-		(property "LCSC part number" "C25879"
+		(property "LCSC" "C25879"
 			(at 36.83 145.415 0)
 			(effects
@@
 			)
 		)
-		(property "LCSC part number" "C381083"
+		(property "LCSC" "C381083"
 			(at 248.92 56.515 0)
 			(effects
@@
 			)
 		)
-		(property "LCSC part number" "C160404"
+		(property "LCSC" "C160404"
 			(at 246.38 134.62 0)
 			(effects
@@
 			)
 		)
-		(property "LCSC part number" "C11702"
+		(property "LCSC" "C11702"
 			(at 78.105 38.1 90)
 			(effects
@@
 			)
 		)
-		(property "LCSC part number" "C64886"
+		(property "LCSC" "C64886"
 			(at 128.905 145.415 90)
 			(effects
@@
 			)
 		)
-		(property "LCSC part number" "C1525"
+		(property "LCSC" "C1525"
 			(at 120.015 156.21 0)
 			(effects
@@
 			)
 		)
-		(property "LCSC part number" "C1525"
+		(property "LCSC" "C1525"
 			(at 219.71 36.83 0)
 			(effects
@@
 			)
 		)
-		(property "LCSC part number" "C25879"
+		(property "LCSC" "C25879"
 			(at 54.61 145.415 0)
 			(effects
@@
 			)
 		)
-		(property "LCSC part number" "C25741"
+		(property "LCSC" "C25741"
 			(at 199.39 45.72 0)
 			(effects
@@
 			)
 		)
-		(property "LCSC part number" "C7420339"
+		(property "LCSC" "C7420339"
 			(at 172.72 46.355 90)
 			(effects
@@
 			)
 		)
-		(property "LCSC part number" "C1525"
+		(property "LCSC" "C1525"
 			(at 86.995 62.23 90)
 			(effects
@@
 			)
 		)
-		(property "LCSC part number" "C381144"
+		(property "LCSC" "C381144"
 			(at 127 52.07 0)
 			(effects
@@
 			)
 		)
-		(property "LCSC part number" "C32346"
+		(property "LCSC" "C32346"
 			(at 100.33 156.21 90)
 			(effects
@@
 			)
 		)
-		(property "LCSC part number" "C11702"
+		(property "LCSC" "C11702"
 			(at 191.135 45.72 0)
 			(effects
@@
 			)
 		)
-		(property "LCSC part number" "C25741"
+		(property "LCSC" "C25741"
 			(at 207.645 45.72 0)
 			(effects
@@
 			)
 		)
-		(property "LCSC part number" "C25741"
+		(property "LCSC" "C25741"
 			(at 215.9 45.72 0)
 			(effects
@@
 			)
 		)
-		(property "LCSC part number" "C25879"
+		(property "LCSC" "C25879"
 			(at 63.5 145.415 0)
 			(effects
@@
 			)
 		)
-		(property "LCSC part number" "C25741"
+		(property "LCSC" "C25741"
 			(at 207.645 65.405 0)
 			(effects
@@
 			)
 		)
-		(property "LCSC part number" "C7464026"
+		(property "LCSC" "C7464026"
 			(at 101.6 54.61 0)
 			(effects

Commit message: Final tweaks after uploading to JLC
Parts:
- C1: footprint Capacitor_SMD:C_0603_1608Metric_Pad1.08x0.95mm_HandSolder -> Capacitor_SMD:C_0603_1608Metric
- D1, D3, D4: footprint Diode_SMD:D_SOD-323_HandSoldering -> Diode_SMD:D_SOD-323
Changed lines of the file:
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@@
 			)
 		)
-		(property "Footprint" "Capacitor_SMD:C_0603_1608Metric_Pad1.08x0.95mm_HandSolder"
+		(property "Footprint" "Capacitor_SMD:C_0603_1608Metric"
 			(at 110.49 156.21 0)
 			(effects
@@
 			)
 		)
-		(property "Footprint" "Diode_SMD:D_SOD-323_HandSoldering"
+		(property "Footprint" "Diode_SMD:D_SOD-323"
 			(at 40.64 48.26 90)
 			(effects
@@
 			)
 		)
-		(property "Footprint" "Diode_SMD:D_SOD-323_HandSoldering"
+		(property "Footprint" "Diode_SMD:D_SOD-323"
 			(at 128.905 134.62 90)
 			(effects
@@
 			)
 		)
-		(property "Footprint" "Diode_SMD:D_SOD-323_HandSoldering"
+		(property "Footprint" "Diode_SMD:D_SOD-323"
 			(at 128.905 145.415 90)
 			(effects
